Commit message: aggiunto nuova telecamera

File: urdf/armando_body.urdf.xacro (robot description, xacro)
@@ -396,4 +396,10 @@
     </joint>
     <link name="camera_mount"/>
+    <!-- <joint name="camera_mount_joint_2" type="fixed">
+        <parent link="crawer_base"/>
+        <child link="second_camera_mount"/>
+        <origin xyz="0.0 0.0 0.0" rpy="1.57079632679 0 0"/>
+    </joint>
+    <link name="second_camera_mount"/> -->
     <!-- ===== Plugin Gazebo ===== -->
     <gazebo>

File: urdf/armando_camera.urdf.xacro (robot description, xacro)
@@ -41,3 +41,43 @@
         </sensor>
     </gazebo>
+    <joint name="camera_joint_2" type="fixed">
+        <parent link="crawer_base"/>
+        <child link="second_camera_link"/>
+        <origin xyz="0.0 0.0 0.0" rpy="0 -1.57079632679 0"/>
+    </joint>
+    <link name="second_camera_link">
+        <visual>
+            <geometry>
+                <box size="0.01 0.03 0.03"/>
+            </geometry>
+            <material name="red"/>
+        </visual>
+    </link>
+    <joint name="second_camera_optical_joint" type="fixed">
+        <parent link="second_camera_link"/>
+        <child link="second_camera_optical_frame"/>
+        <origin xyz="0 0 0" rpy="-1.57079632679 0 -1.57079632679"/>
+    </joint>
+    <link name="second_camera_optical_frame"/>
+    <!-- ==== Plugin Sensore ==== -->
+    <gazebo reference="second_camera_link">
+        <sensor name="second_camera" type="camera">
+            <camera>
+                <horizontal_fov>1.047</horizontal_fov>
+                <image>
+                    <width>1920</width>
+                    <height>1080</height>
+                </image>
+                <clip>
+                    <near>0.1</near>
+                    <far>5</far>
+                </clip>
+            </camera>
+            <always_on>1</always_on>
+            <update_rate>30</update_rate>
+            <visualize>true</visualize>
+            <topic>second_camera</topic>
+            <gz_frame_id>second_camera_optical_frame</gz_frame_id>
+        </sensor>
+    </gazebo>
 </robot>
